File: MCU_Datalogger.kicad_sch (KiCad schematic)
At the start: 25 parts, among them U1 24LC1025, U2 DS1337S_, U3 24LC1025, U4 ATMEGA328P-AU, Y1 32.768 KHz, Y2 16 MHz

Commit message: Completed comments.
Connections:
- no-connect marks 8 -> 9
Other:
- sheet Connectors ports: added D2, D3, D4, D5, D6, D7, D8, GND, MISO, MOSI, RESET, RX, SCK, SDA, TX, VCC; removed none
- note added: "EEPROM"
- note added: "MCU"
- note added: "Mounting"
- note added: "Real Time Clock"
- moved on the sheet: BAT1, C1, C2, C3, C4, C5, D1, D2, H1, H2, H3, H4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

Commit message: Completed routing.
Connections:
- net GND: now also BAT1.2; no longer BAT1.Neg
- net at C5.1, D2.2 (A), U4.18 (AVCC)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: now also BAT1.1; no longer BAT1.Pos
Changed lines of the file:
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@@
 			)
 		)
-		(pin "Neg"
+		(property "Purpose" ""
+			(at 267.97 44.45 0)
+			(effects
+				(font
+					(size 1.27 1.27)
+				)
+			)
 		)
-		(pin "Pos"
+		(pin "2"
+		)
+		(pin "1"
 		)
 		(instances

Commit message: Completed the Design.
Connections:
- net VCC: now also BAT1.1, C5.1, D2.2 (A), U4.18 (AVCC), U4.4 (VCC)
Changed lines of the file:
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@@
+		)
+	)
+	(label "VCC"
+		(at 260.35 39.37 0)
+		(effects
+			(font
+				(size 1.27 1.27)
+			)
+			(justify left bottom)
 		)
 	)

Commit message: Fixed two defects in the schematic.
Connections:
- net SCK: no longer U1.6 (SCL), U2.6 (SCL), U3.6 (SCL), U4.28 (PC5)
- new net SCL: U1.6 (SCL), U2.6 (SCL), U3.6 (SCL), U4.28 (PC5)
Other:
- sheet Connectors ports: added SCL; removed none
Changed lines of the file:
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@@
 	)
 	(junction
-		(at 101.6 40.64)
-		(diameter 0)
-		(color 0 0 0 0)
-	)
-	(junction
 		(at 243.84 39.37)
 		(diameter 0)
@@
 	(wire
 		(pts
-			(xy 97.79 40.64) (xy 101.6 40.64)
-		)
-		(stroke
-			(width 0)
-			(type default)
-		)
-	)
-	(wire
-		(pts
 			(xy 224.79 85.09) (xy 228.6 85.09)
 		)
@@
 	(wire
 		(pts
-			(xy 101.6 40.64) (xy 111.76 40.64)
+			(xy 97.79 40.64) (xy 111.76 40.64)
 		)
 		(stroke
@@
 		)
 	)
-	(label "SCK"
+	(label "SCL"
 		(at 50.8 52.07 180)
 		(effects
@@
 		)
 	)
-	(label "SCK"
+	(label "SCL"
 		(at 181.61 129.54 180)
 		(effects
@@
 		)
 	)
-	(label "SCK"
+	(label "SCL"
 		(at 66.04 143.51 0)
 		(effects
@@
 		)
 	)
-	(label "SCK"
+	(label "SCL"
 		(at 102.87 143.51 0)
 		(effects
@@
 		)
 	)
-	(label "SCK"
+	(label "SCL"
 		(at 194.31 82.55 180)
 		(effects
@@
 		)
 	)
+	(label "SCK"
+		(at 181.61 143.51 180)
+		(effects
+			(font
+				(size 1.27 1.27)
+			)
+			(justify right bottom)
+		)
+	)
 	(label "D5"
 		(at 215.9 130.81 0)
@@
 	)
 	(symbol
-		(lib_id "power:PWR_FLAG")
-		(at 101.6 40.64 0)
-		(unit 1)
-		(exclude_from_sim no)
-		(in_bom yes)
-		(on_board yes)
-		(dnp no)
-		(fields_autoplaced yes)
-		(property "Reference" "#FLG01"
-			(at 101.6 38.735 0)
-			(effects
-				(font
-					(size 1.27 1.27)
-				)
-				(hide yes)
-			)
-		)
-		(property "Value" "PWR_FLAG"
-			(at 101.6 36.195 0)
-			(effects
-				(font
-					(size 1.27 1.27)
-				)
-			)
-		)
-		(property "Footprint" ""
-			(at 101.6 40.64 0)
-			(effects
-				(font
-					(size 1.27 1.27)
-				)
-				(hide yes)
-			)
-		)
-		(property "Datasheet" "~"
-			(at 101.6 40.64 0)
-			(effects
-				(font
-					(size 1.27 1.27)
-				)
-				(hide yes)
-			)
-		)
-		(property "Description" "Special symbol for telling ERC where power comes from"
-			(at 101.6 40.64 0)
-			(effects
-				(font
-					(size 1.27 1.27)
-				)
-				(hide yes)
-			)
-		)
-		(pin "1"
-		)
-		(instances
-			(project ""
-				(path "/be1eed37-8a6f-4061-89c1-54ae666185b6"
-					(reference "#FLG01")
-					(unit 1)
-				)
-			)
-		)
-	)
-	(symbol
 		(lib_id "power:GND")
 		(at 179.07 118.11 0)
@@
 			)
 		)
-		(pin "SCK" passive
-			(at 181.61 129.54 180)
-			(effects
-				(font
-					(size 1.27 1.27)
-				)
-				(justify left)
-			)
-		)
 		(pin "RX" input
 			(at 181.61 140.97 180)
@@
 			(effects
 				(font
+					(size 1.27 1.27)
+				)
+				(justify left)
+			)
+		)
+		(pin "SCK" passive
+			(at 181.61 143.51 180)
+			(effects
+				(font
+					(size 1.27 1.27)
+				)
+				(justify left)
+			)
+		)
+		(pin "SCL" passive
+			(at 181.61 129.54 180)
+			(effects
+				(font

Commit message: Fixed all defects.
Connections:
- net SCK: no longer R3.2
- net SCL: now also R3.2
Changed lines of the file:
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@@
 		)
 	)
-	(label "SCK"
+	(label "SCL"
 		(at 118.11 153.67 180)
 		(effects
